Commit message: updating model files

File: atlas_description/urdf/atlas_unplugged_v5_dual_robotiq_with_head_mod_34.urdf (robot description, URDF)
Before this commit: robot atlas, 75 links, 74 joints
Links:
- link l_foot: geometry collision box size=0.195 0.133887 0.05; visual box size=0.195 0.133887 0.05
- link l_toe: geometry collision box size=0.065 0.133887 0.05; visual box size=0.065 0.133887 0.05
- link r_foot: geometry collision box size=0.195 0.133887 0.05; visual box size=0.195 0.133887 0.05
- link r_toe: geometry collision box size=0.065 0.133887 0.05; visual box size=0.065 0.133887 0.05
Joints:
- joint l_leg_toe: origin xyz=0.042 0 -0.05 rpy=0 0 0 -> xyz=0.107 0 -0.05 rpy=0 0 0
- joint r_leg_toe: origin xyz=0.042 0 -0.05 rpy=0 0 0 -> xyz=0.107 0 -0.05 rpy=0 0 0
